File: kicad/lab8.kicad_sch (KiCad schematic)
At the start: 44 parts, among them Q1 LTR3208E, SW1 Reset, U2 74xxx244, U3 MCP6294, U4 PIC32MX170F256B, U5 LM339AN

Commit message: Annotate IR receiver schematic
Parts:
- removed C?: 0.1uF, symbol ME218_BaseLib:Cap
- C?: value 0.001uF -> 1nF
- R? (x2): value 10K -> 20k
Other:
- note added: "Stage 1: current to voltage"
- note added: "Stage 2: filter high frequency noise"
- note added: "Stage 3: spike up or down"
- note added: "Stage 4: square wave"
- moved on the sheet: C2, C3, C4, C5, C6, C7, C8, C9, C?, PRG1, Q1, Q?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
